File: pcb/Example_from_KiCad-Template_LED.kicad_pcb (KiCad board)
At the start: 2 copper layers, 80 x 50 mm, 5 parts

Commit message: PCB created
Parts:
- added BT1: 3V, Battery:BatteryHolder_Keystone_1060_1x2032, F.Cu at (137.3, 94.5)
- added D1: LED, LED_THT:LED_D5.0mm, F.Cu at (146.3, 108.8)
- added R1: 1k, TIH:R_axial_SMD-Adapter_P10.16mm_1mm, F.Cu at (122.1, 108.8)
Routing:
- net Net-(BT1-+): track 0.00 -> 16.6 mm
- net Net-(BT1--): track 0.00 -> 16.6 mm
- net Net-(D1-A): track 0.00 -> 11.5 mm
Other:
- board text added: "PCB-LED Example from KiCad-Template HTL-Rankweil 9/2026 TIH"
